Commit message: finally setup

File: hb_robot_control/urdf/hb_robot_controlled.urdf.xacro (robot description, xacro)
@@ -4,9 +4,8 @@
     <xacro:include filename="$(find ur_description)/urdf/ur.ros2_control.xacro"/>
     <xacro:arg name="ur_type" default="ur10e"/>
-    <xacro:arg name="joint_limits_parameters_file" default="$(find ur_description)/config/$(arg ur_type)/joint_limits.yaml"/>
-    <xacro:arg name="kinematics_parameters_file" default="$(find hb_robot_description)/urdf/my_robot_calibration.yaml"/>
-    <xacro:arg name="kinematics_hash" default="calib_16746413789305179772"/>
-    <xacro:arg name="physical_parameters_file" default="$(find ur_description)/config/$(arg ur_type)/physical_parameters.yaml"/>
-    <xacro:arg name="visual_parameters_file" default="$(find ur_description)/config/$(arg ur_type)/visual_parameters.yaml"/>
+    <xacro:arg name="joint_limit_params" default="$(find hb_robot_control)/config/$(arg ur_type)/joint_limits.yaml"/>
+    <xacro:arg name="kinematics_params" default="$(find hb_robot_control)/config/$(arg ur_type)/default_kinematics.yaml"/>
+    <xacro:arg name="physical_params" default="$(find hb_robot_control)/config/$(arg ur_type)/physical_parameters.yaml"/>
+    <xacro:arg name="visual_params" default="$(find hb_robot_control)/config/$(arg ur_type)/visual_parameters.yaml"/>
     <xacro:arg name="robot_ip" default="192.168.200.55"/>
     <xacro:arg name="headless_mode" default="false" />
@@ -14,28 +13,30 @@
     <xacro:arg name="ur_output_recipe_filename" default="$(find ur_robot_driver)/resources/rtde_output_recipe.txt"/>
     <xacro:arg name="ur_input_recipe_filename" default="$(find ur_robot_driver)/resources/rtde_input_recipe.txt"/>
-    <xacro:arg name="use_mock_hardware" default="false" />
-    <xacro:arg name="mock_sensor_commands" default="false" />
+    <xacro:arg name="use_fake_hardware" default="false" />
+    <xacro:arg name="fake_sensor_commands" default="false" />
+    <xacro:property name="kinematics_params_file" value="$(arg kinematics_params)"/>
+    <xacro:property name="kinematics_hash" value="${xacro.load_yaml(kinematics_params_file)['kinematics']['hash']}"/>
     <link name="world"/>
     <xacro:hb_robot
         parent="world"
         ur_type="$(arg ur_type)"
-        joint_limits_parameters_file="$(arg joint_limits_parameters_file)"
-        kinematics_parameters_file="$(arg kinematics_parameters_file)"
-        physical_parameters_file="$(arg physical_parameters_file)"
-        visual_parameters_file="$(arg visual_parameters_file)"
+        joint_limits_parameters_file="$(arg joint_limit_params)"
+        kinematics_parameters_file="$(arg kinematics_params)"
+        physical_parameters_file="$(arg physical_params)"
+        visual_parameters_file="$(arg visual_params)"
         >
       <origin xyz="0 0 0" rpy="0 0 0" />
     </xacro:hb_robot>
     <!--Create the control tag for the UR robot-->
-    <xacro:ur_ros2_control
-      name="my_$(arg ur_type)"
+      <xacro:ur_ros2_control
+      name="$(arg ur_type)"
       tf_prefix="$(arg ur_type)_"
+      hash_kinematics="${kinematics_hash}"
       robot_ip="$(arg robot_ip)"
-      hash_kinematics= "$(arg kinematics_hash)"
       script_filename="$(arg ur_script_filename)"
       output_recipe_filename="$(arg ur_output_recipe_filename)"
       input_recipe_filename="$(arg ur_input_recipe_filename)"
-      use_fake_hardware="$(arg use_mock_hardware)"
-      fake_sensor_commands="$(arg mock_sensor_commands)"
+      use_fake_hardware="$(arg use_fake_hardware)"
+      fake_sensor_commands="$(arg fake_sensor_commands)"
       headless_mode="$(arg headless_mode)"
     />

File: hb_robot_description/urdf/hb_robot_macro.xacro (robot description, xacro)
@@ -44,4 +44,5 @@
             physical_parameters_file="${physical_parameters_file}"
             visual_parameters_file="${visual_parameters_file}"
+            generate_ros2_control_tag="false"
             >
             <origin xyz="0 0 0" rpy="${pi/2} 0 0" />
