Commit message: random

File: hb_robot_description/urdf/hb_sensors_macro.xacro (robot description, xacro)
@@ -6,5 +6,5 @@
     <parent link="${ur_type}_tool0"/>
     <child link="camera_base"/>
-    <origin xyz= "0.05 0.07 0.06" rpy="0.002 -0.001 -2.36"/>
+    <origin xyz= "0.1 0.1 0.1" rpy="${pi} -${pi/2} 0"/>
 </joint>
 <!-- <link name="unilidar_lidar"/> -->
@@ -18,5 +18,5 @@
     <parent link="robot_mount"/>
     <child link= "unilidar_imu_initial"/>
-    <origin xyz="1 1 0" rpy="0 0 0"/>
+    <origin xyz="0 0 1.1" rpy="${pi/2} 0 0"/>
 </joint>
 </xacro:macro>
