Commit message: update lots

File: hb_robot_description/urdf/hb_sensors_macro.xacro (robot description, xacro)
@@ -16,7 +16,7 @@
 </joint> -->
 <joint name="mount_to_imu" type="fixed">
-    <parent link="robot_mount"/>
+    <parent link="HB_carriage"/>
     <child link= "unilidar_imu_initial"/>
-    <origin xyz="0 0 1.1" rpy="${pi/2} 0 0"/>
+    <origin xyz="0 0 1.1" rpy="0 0 ${pi}"/>
 </joint>
 </xacro:macro>

Commit message: bringup for ur10e

File: hb_robot_description/urdf/hb_sensors_macro.xacro (robot description, xacro)
@@ -2,10 +2,10 @@
 <robot xmlns:xacro="http://www.ros.org/wiki/xacro">
 <xacro:macro name="hb_sensors" params="ur_type">
-<xacro:include filename="$(find azure_kinect_ros2_driver)/urdf/azure_kinect.urdf.xacro"/>
-<joint name="tool0_to_kinect" type="fixed">
+<!-- <xacro:include filename="$(find azure_kinect_ros2_driver)/urdf/azure_kinect.urdf.xacro"/> -->
+<!-- <joint name="tool0_to_kinect" type="fixed">
     <parent link="${ur_type}_tool0"/>
     <child link="camera_base"/>
     <origin xyz= "0.1 0.1 0.1" rpy="${pi} -${pi/2} 0"/>
-</joint>
+</joint> -->
 <!-- <link name="unilidar_lidar"/> -->
 <link name="unilidar_imu_initial"/>

Commit message: azure sorted

File: hb_robot_description/urdf/hb_sensors_macro.xacro (robot description, xacro)
@@ -2,12 +2,12 @@
 <robot xmlns:xacro="http://www.ros.org/wiki/xacro">
 <xacro:macro name="hb_sensors" params="ur_type">
-<!-- <xacro:include filename="$(find azure_kinect_ros2_driver)/urdf/azure_kinect.urdf.xacro"/> -->
-<!-- <joint name="tool0_to_kinect" type="fixed">
+<xacro:include filename="$(find azure_kinect_ros2_driver)/urdf/azure_kinect.urdf.xacro"/>
+<joint name="tool0_to_kinect" type="fixed">
     <parent link="${ur_type}_tool0"/>
     <child link="camera_base"/>
     <origin xyz= "0.1 0.1 0.1" rpy="${pi} -${pi/2} 0"/>
-</joint> -->
+</joint>
 <!-- <link name="unilidar_lidar"/> -->
-<link name="unilidar_imu_initial"/>
+<!-- <link name="unilidar_imu_initial"/> -->
 <!-- <joint name="mount_to_lidar" type="fixed">
     <parent link="robot_mount"/>
@@ -15,9 +15,9 @@
     <origin xyz="1 0 0" rpy="0 0 0"/>
 </joint> -->
-<joint name="mount_to_imu" type="fixed">
+<!--<joint name="mount_to_imu" type="fixed">
     <parent link="HB_carriage"/>
     <child link= "unilidar_imu_initial"/>
     <origin xyz="0 0 1.1" rpy="0 0 ${pi}"/>
-</joint>
+</joint> -->
 </xacro:macro>
 </robot>

Commit message: calibrated camera, changed qos

File: hb_robot_description/urdf/hb_sensors_macro.xacro (robot description, xacro)
@@ -3,8 +3,13 @@
 <xacro:macro name="hb_sensors" params="ur_type">
 <xacro:include filename="$(find azure_kinect_ros2_driver)/urdf/azure_kinect.urdf.xacro"/>
-<joint name="tool0_to_kinect" type="fixed">
+<!-- <joint name="tool0_to_kinect" type="fixed">
     <parent link="${ur_type}_tool0"/>
     <child link="camera_base"/>
     <origin xyz= "-0.125 0 .15" rpy="0 ${-pi/2} 0"/>
+</joint> -->
+<joint name="calibrated_camera_mount" type="fixed">
+  <parent link="${ur_type}_tool0"/>
+  <child link="camera_base"/>
+  <origin xyz="-0.05878718188937343 0.059510573280679324 0.1513621946385637" rpy="-1.56712649894296 -0.7779397496579974 1.5852325385326869"/>
 </joint>
 <!-- <link name="unilidar_lidar"/> -->

Commit message: added unilidar

File: hb_robot_description/urdf/hb_sensors_macro.xacro (robot description, xacro)
@@ -13,6 +13,6 @@
   <origin xyz="-0.05878718188937343 0.059510573280679324 0.1513621946385637" rpy="-1.56712649894296 -0.7779397496579974 1.5852325385326869"/>
 </joint>
-<!-- <link name="unilidar_lidar"/> -->
-<!-- <link name="unilidar_imu_initial"/> -->
+<link name="unilidar_lidar"/>
+<link name="unilidar_imu"/>
 <!-- <joint name="mount_to_lidar" type="fixed">
     <parent link="robot_mount"/>
@@ -20,9 +20,15 @@
     <origin xyz="1 0 0" rpy="0 0 0"/>
 </joint> -->
-<!--<joint name="mount_to_imu" type="fixed">
+<joint name="mount_to_imu" type="fixed">
     <parent link="HB_carriage"/>
-    <child link= "unilidar_imu_initial"/>
-    <origin xyz="0 0 1.1" rpy="0 0 ${pi}"/>
-</joint> -->
+    <child link= "unilidar_lidar"/>
+    <origin xyz="-.1425 0 .544" rpy="${-pi/2} ${(pi/8) -(pi/2)} 0"/>
+</joint>
+<joint name="lidar_to_imu" type="fixed">
+    <parent link="unilidar_lidar"/>
+    <child link="unilidar_imu"/>
+    <origin xyz="-0.007698 -0.014655 0.006670"
+            rpy="0 0 0"/>
+</joint>
 </xacro:macro>
 </robot>
