Commit message: rewriting the exploration planning skill

File: hb_robot_description/urdf/hb_robot_macro.xacro (robot description, xacro)
@@ -48,4 +48,43 @@
             <origin xyz="0 0 0" rpy="${pi/2} 0 0" />
         </xacro:ur_robot>
+        <!-- END EFFECTOR STUFF -->
+        <link name="${ur_type}_bracket_link">
+            <visual>
+                <geometry>
+                <mesh filename="package://hb_robot_description/meshes/bracket.stl"/>
+                </geometry>
+                <origin rpy="0 0 0" xyz="0 0 0"/>
+            </visual>
+            <collision>
+                <geometry>
+                <mesh filename="package://hb_robot_description/meshes/bracket.stl"/>
+                </geometry>
+                <origin rpy="0 0 0" xyz="0 0 0"/>
+            </collision>
+        </link>
+        <joint name="eef_bracket_joint" type="fixed">
+            <parent link="${ur_type}_tool0" />
+            <child link="${ur_type}_bracket_link" />
+            <origin xyz= "0 0 0" rpy="0 0 ${pi}"/>
+        </joint>
+        <link name="${ur_type}_torch_link">
+            <visual>
+                <geometry>
+                <mesh filename="package://hb_robot_description/meshes/torch.stl"/>
+                </geometry>
+                <origin rpy="0 0 0" xyz="0 0 0"/>
+            </visual>
+            <collision>
+                <geometry>
+                <mesh filename="package://hb_robot_description/meshes/torch.stl"/>
+                </geometry>
+                <origin rpy="0 0 0" xyz="0 0 0"/>
+            </collision>
+        </link>
+        <joint name="eef_bracket_torch_joint" type="fixed">
+            <parent link="${ur_type}_bracket_link" />
+            <child link="${ur_type}_torch_link" />
+            <origin xyz= "-.04415 0.00146 0.48478" rpy="2.3562 -0.0007 ${pi+0.0004}"/>
+        </joint>
     </xacro:macro>
 </robot>

File: hb_robot_description/urdf/hb_sensors_macro.xacro (robot description, xacro)
@@ -6,5 +6,5 @@
     <parent link="${ur_type}_tool0"/>
     <child link="camera_base"/>
-    <origin xyz= "0.1 0.1 0.1" rpy="${pi} -${pi/2} 0"/>
+    <origin xyz= "-0.125 0 .15" rpy="0 ${-pi/2} 0"/>
 </joint>
 <!-- <link name="unilidar_lidar"/> -->
