Commit message: homing_routine

File: crane_description/urdf/crane/crane_macro.ros2_control.xacro (robot description, xacro)
@@ -17,4 +17,10 @@
         <param name="right_steps_per_unit">1000.0</param>
       </hardware>
+      <gpio name="crane">
+        <command_interface name="home"/>
+        <state_interface name="homing"/>
+        <state_interface name="homed"/>
+        <state_interface name="home_failed"/>
+      </gpio>
       <joint name="swivel_joint">
         <command_interface name="position"/>

File: crane_description/urdf/crane/crane_macro.xacro (robot description, xacro)
@@ -23,5 +23,5 @@
             <origin xyz="0 0 0" rpy="0 0 0"/>
             <geometry>
-                <cylinder size= "0.05 0.1"/>
+                <cylinder radius="0.05" length="0.1"/>
             </geometry>
             </collision>
@@ -29,5 +29,5 @@
             <origin xyz="0 0 0" rpy="0 0 0"/>
             <geometry>
-                <cylinder size= "0.05 0.1"/>
+                <cylinder radius="0.05" length="0.1"/>
             </geometry>
             <material name="light_red"/>
@@ -38,5 +38,5 @@
             <origin xyz="0 0 0" rpy="0 0 0"/>
             <geometry>
-                <cylinder size= "0.05 0.1"/>
+                <cylinder radius="0.05" length="0.1"/>
             </geometry>
             </collision>
@@ -44,5 +44,5 @@
             <origin xyz="0 0 0" rpy="0 0 0"/>
             <geometry>
-                <cylinder size= "0.05 0.1"/>
+                <cylinder radius="0.05" length="0.1"/>
             </geometry>
             <material name="light_red"/>

Commit message: add extra interfaces to control xacro

File: crane_description/urdf/crane/crane_macro.ros2_control.xacro (robot description, xacro)
@@ -19,4 +19,10 @@
         <param name="g1_steps_per_unit">25.0</param>
       </hardware>
+      <gpio name="G0_wheels">
+        <command_interface name="velocity"/>
+      </gpio>
+      <gpio name="G1_wheels">
+        <command_interface name="velocity"/>
+      </gpio>
       <gpio name="crane">
         <command_interface name="home"/>
@@ -37,23 +43,24 @@
         <state_interface name="position"/>
       </joint>
-<!--
-      <joint name="swivel_joint">
-        <command_interface name="velocity"/>
+      <joint name="G0_joint">
         <command_interface name="position"/>
-        <state_interface name="velocity"/>
         <state_interface name="position"/>
       </joint>
-      <joint name="LG_lin_joint">
-        <command_interface name="velocity"/>
+      <joint name="G1_joint">
         <command_interface name="position"/>
-        <state_interface name="velocity"/>
         <state_interface name="position"/>
       </joint>
-      <joint name="RG_lin_joint">
-        <command_interface name="velocity"/>
-        <command_interface name="position"/>
+      <joint name="w0_joint">
         <state_interface name="velocity"/>
-        <state_interface name="position"/>
-      </joint> -->
+      </joint>
+      <joint name="w1_joint">
+        <state_interface name="velocity"/>
+      </joint>
+      <joint name="w2_joint">
+        <state_interface name="velocity"/>
+      </joint>
+      <joint name="w3_joint">
+        <state_interface name="velocity"/>
+      </joint>
     </ros2_control>
   </xacro:macro>
