Commit message: adjusted

File: crane_description/urdf/crane/crane_macro.xacro (robot description, xacro)
@@ -34,4 +34,5 @@
             </visual>
         </link>
+        <link name="Crane_RS_link"/>
         <link name="LG_link">
             <collision>
@@ -85,4 +86,9 @@
             <limit lower="0.0" upper="0.5" effort="100" velocity="1.0"/>
         </joint>
+        <joint name="spreader_camera_joint" type="fixed">
+            <parent link="spreader_link"/>
+            <child link ="Crane_RS_link"/>
+            <origin xyz ="0 0 0" rpy="0 0 0"/>
+        </joint>
     </xacro:macro>
 </robot>

Commit message: updated crane urdf

File: crane_description/urdf/crane/crane_macro.xacro (robot description, xacro)
@@ -49,15 +49,28 @@
             </visual>
         </link>
-        <link name="spreader_link">
-            <collision>
-            <origin xyz="0 0 0" rpy="0 0 0"/>
-            <geometry>
-                <box size= "1 0.08 0.08"/>
-            </geometry>
-            </collision>
-            <visual>
-            <origin xyz="0 0 0" rpy="0 0 0"/>
-            <geometry>
-                <box size= "1 0.08 0.08"/>
+        <link name="chassis_link">
+            <inertial>
+             <origin
+                xyz="0.00317 -0.01646 0.0625"
+                rpy="0 0 0" />
+            <mass value="44.667"/>
+            <inertia
+                ixx="16.383145"
+                ixy="-0.02317"
+                ixz="-0.013012"
+                iyy="0.949633"
+                iyz="0.77285"
+                izz="16.145575"/>
+            </inertial>
+            <collision>
+            <origin xyz="0 0 0" rpy="0 0 0"/>
+            <geometry>
+                <mesh filename="package://crane_description/meshes/chassis.stl"/>
+            </geometry>
+            </collision>
+            <visual>
+            <origin xyz="0 0 0" rpy="0 0 0"/>
+            <geometry>
+                <mesh filename="package://crane_description/meshes/chassis.stl"/>
             </geometry>
             <material name="light_red"/>
@@ -96,4 +109,12 @@
             </visual>
         </link>
+        <link name="Gimbal_0_link"/>
+        <link name="Gimbal_1_link"/>
+        <link name="Gimbal_2_link"/>
+        <link name="Gimbal_3_link"/>
+        <link name="w0_link"/>
+        <link name="w1_link"/>
+        <link name="w2_link"/>
+        <link name="w3_link"/>
         <joint name="base_sw_top_joint" type = "fixed">
             <parent link="base_link"/>
@@ -110,6 +131,6 @@
         <joint name="swivel_spreader_joint" type="fixed">
             <parent link="swivel_bottom"/>
-            <child link="spreader_link"/>
-            <origin xyz="0 0 -0.75" rpy="0 0 0"/>
+            <child link="chassis_link"/>
+            <origin xyz="0 0 -0.835" rpy="0 0 0"/>
         </joint>
         <joint name="swivel_bottom_tag_joint" type="fixed">
@@ -119,22 +140,80 @@
         </joint>
         <joint name="LG_lin_joint" type="prismatic">
-            <parent link="spreader_link"/>
+            <parent link="chassis_link"/>
             <child link="LG_link"/>
-            <origin xyz="-0.25 0 -0.08" rpy="0 0 0"/>
-            <axis xyz="1 0 0"/>
+            <origin xyz="0 -0.5 -0.191" rpy="0 0 0"/>
+            <axis xyz="0 1 0"/>
             <limit lower="-0.5" upper="0.0" effort="100" velocity="1.0"/>
         </joint>
         <joint name="RG_lin_joint" type="prismatic">
-            <parent link="spreader_link"/>
+            <parent link="chassis_link"/>
             <child link="RG_link"/>
-            <origin xyz="0.25 0 -0.08" rpy="0 0 0"/>
-            <axis xyz="1 0 0"/>
+            <origin xyz="0 -0.5 -0.191" rpy="0 0 0"/>
+            <axis xyz="0 1 0"/>
             <limit lower="0.0" upper="0.5" effort="100" velocity="1.0"/>
         </joint>
         <joint name="spreader_RS_joint" type="fixed">
-            <parent link="spreader_link"/>
+            <parent link="chassis_link"/>
             <child link ="Crane_RS_link"/>
             <origin xyz ="0 0 0" rpy="0 0 0"/>
         </joint>
+        <joint name="G0_joint" type="revolute">
+            <parent link="chassis_link"/>
+            <child link="Gimbal_0_link"/>
+            <origin xyz="0.125 0.3595 0.155" rpy="0 0 0"/>
+            <axis xyz="1 0 0"/>
+            <limit lower="-1.57" upper="1.57" effort="100" velocity="1.0"/>
+        </joint>
+        <joint name="G3_joint" type="revolute">
+            <parent link="chassis_link"/>
+            <child link="Gimbal_3_link"/>
+            <origin xyz="0.125 -0.3595 0.155" rpy="0 0 0"/>
+            <axis xyz="1 0 0"/>
+            <mimic joint="G0_joint" multiplier="-1" offset="0.0"/>
+            <limit lower="-1.57" upper="1.57" effort="100" velocity="1.0"/>
+        </joint>
+        <joint name="G1_joint" type="revolute">
+            <parent link="chassis_link"/>
+            <child link="Gimbal_1_link"/>
+            <origin xyz="-0.0005 0.115 0.28" rpy="0 0 0"/>
+            <axis xyz="0 0 1"/>
+            <limit lower="-1.57" upper="1.57" effort="100" velocity="1.0"/>
+        </joint>
+        <joint name="G2_joint" type="revolute">
+            <parent link="chassis_link"/>
+            <child link="Gimbal_2_link"/>
+            <origin xyz="-0.0005 -0.115 0.28" rpy="0 0 0"/>
+            <axis xyz="0 0 1"/>
+            <mimic joint="G1_joint" multiplier="-1" offset="0.0"/>
+            <limit lower="-1.57" upper="1.57" effort="100" velocity="1.0"/>
+        </joint>
+        <joint name="w0_joint" type="continuous">
+            <parent link="Gimbal_0_link"/>
+            <child link="w0_link"/>
+            <origin xyz="-0.125 0 0" rpy="0 0 0"/>
+            <axis xyz="0 1 0"/>
+            <limit effort="100" velocity="1.0"/>
+        </joint>
+        <joint name="w1_joint" type="continuous">
+            <parent link="Gimbal_1_link"/>
+            <child link="w1_link"/>
+            <origin xyz="0 0 -0.125" rpy="0 0 0"/>
+            <axis xyz="1 0 0"/>
+            <limit effort="100" velocity="1.0"/>
+        </joint>
+        <joint name="w2_joint" type="continuous">
+            <parent link="Gimbal_2_link"/>
+            <child link="w2_link"/>
+            <origin xyz="0 0 -0.125" rpy="0 0 0"/>
+            <axis xyz="1 0 0"/>
+            <limit effort="100" velocity="1.0"/>
+        </joint>
+        <joint name="w3_joint" type="continuous">
+            <parent link="Gimbal_3_link"/>
+            <child link="w3_link"/>
+            <origin xyz="-0.125 0 0" rpy="0 0 0"/>
+            <axis xyz="0 1 0"/>
+            <limit effort="100" velocity="1.0"/>
+        </joint>
     </xacro:macro>
 </robot>

Commit message: fixed posestamped

File: crane_description/urdf/crane/crane_macro.xacro (robot description, xacro)
@@ -78,5 +78,7 @@
         </link>
         <link name = "Swivel_Tag"/>
-        <link name="Crane_RS_link"/>
+        <link name="Trolley_link"/>
+        <link name="Spreader_RS_link"/>
+        <link name="Trolley_RS_link"/>
         <link name="LG_link">
             <collision>
@@ -371,5 +373,15 @@
         <joint name="spreader_RS_joint" type="fixed">
             <parent link="chassis_link"/>
-            <child link ="Crane_RS_link"/>
+            <child link ="Spreader_RS_link"/>
+            <origin xyz ="0 0 0" rpy="0 0 0"/>
+        </joint>
+        <joint name="base_trolley_joint" type="fixed">
+            <parent link="base_link"/>
+            <child link ="Trolley_link"/>
+            <origin xyz ="0 0 0" rpy="0 0 0"/>
+        </joint>
+        <joint name="trolley_RS_joint" type="fixed">
+            <parent link="Trolley_link"/>
+            <child link ="Trolley_RS_link"/>
             <origin xyz ="0 0 0" rpy="0 0 0"/>
         </joint>
