Commit message: fuck this is complicated

File: crane_description/urdf/crane/spreader_macro.xacro (robot description, xacro)
@@ -3,4 +3,5 @@
      <xacro:macro name="spreader">
         <!-- LINKS -->
+        <link name="left_spreader_pose"/>
         <link name="chassis_link">
             <inertial>
@@ -363,4 +364,9 @@
             <limit effort="100" velocity="1.0"/>
         </joint>
+        <joint name="tag_chassis" type="fixed">
+            <child link="chassis_link"/>
+            <parent link="left_spreader_pose"/>
+            <origin xyz="0 -0.5 -0.191" rpy="0 0 0"/>
+        </joint>
     </xacro:macro>
 </robot>

Commit message: estimator  package

File: crane_description/urdf/crane/spreader_macro.xacro (robot description, xacro)
@@ -4,4 +4,5 @@
         <!-- LINKS -->
         <link name="left_spreader_pose"/>
+        <link name="right_spreader_pose"/>
         <link name="chassis_link">
             <inertial>
@@ -364,8 +365,13 @@
             <limit effort="100" velocity="1.0"/>
         </joint>
-        <joint name="tag_chassis" type="fixed">
-            <child link="chassis_link"/>
-            <parent link="left_spreader_pose"/>
-            <origin xyz="0 -0.5 -0.191" rpy="0 0 0"/>
+        <joint name="left_tag_chassis_joint" type="fixed">
+            <parent link="chassis_link"/>
+            <child link="left_spreader_pose"/>
+            <origin xyz=".125 -0.6745 0.363" rpy="0 0 0"/>
+        </joint>
+        <joint name="right_tag_chassis_joint" type="fixed">
+            <parent link="chassis_link"/>
+            <child link="right_spreader_pose"/>
+            <origin xyz=".125 0.6745 0.363" rpy="0 0 0"/>
         </joint>
     </xacro:macro>
