Commit message: adjusted crane trolley pose

File: crane_description/urdf/crane/trolley_macro.xacro (robot description, xacro)
@@ -7,5 +7,5 @@
             <parent link="base_link"/>
             <child link ="Trolley_link"/>
-            <origin xyz ="0 0 0" rpy="0 0 0"/>
+            <origin xyz ="0 0 0" rpy="${-pi} 0 ${-pi/2}"/>
         </joint>
     <link name="Trolley_RS_link"/>
