Commit message: fixed urdf

File: crane_description/urdf/common.xacro (robot description, xacro)
@@ -17,3 +17,6 @@
         <color rgba="${200/255} ${10/255} ${10/255} 1.0"/>
     </material>
+    <material name= "light_blue">
+        <color rgba="${10/255} ${10/255} ${200/255} 1.0"/>
+    </material>
 </robot>

File: crane_description/urdf/crane/crane_macro.xacro (robot description, xacro)
@@ -19,4 +19,34 @@
             </visual>
         </link>
+        <link name = "swivel_top">
+            <collision>
+            <origin xyz="0 0 0" rpy="0 0 0"/>
+            <geometry>
+                <cylinder size= "0.05 0.1"/>
+            </geometry>
+            </collision>
+            <visual>
+            <origin xyz="0 0 0" rpy="0 0 0"/>
+            <geometry>
+                <cylinder size= "0.05 0.1"/>
+            </geometry>
+            <material name="light_red"/>
+            </visual>
+        </link>
+        <link name = "swivel_bottom">
+            <collision>
+            <origin xyz="0 0 0" rpy="0 0 0"/>
+            <geometry>
+                <cylinder size= "0.05 0.1"/>
+            </geometry>
+            </collision>
+            <visual>
+            <origin xyz="0 0 0" rpy="0 0 0"/>
+            <geometry>
+                <cylinder size= "0.05 0.1"/>
+            </geometry>
+            <material name="light_red"/>
+            </visual>
+        </link>
         <link name="spreader_link">
             <collision>
@@ -34,4 +64,5 @@
             </visual>
         </link>
+        <link name = "Swivel_Tag"/>
         <link name="Crane_RS_link"/>
         <link name="LG_link">
@@ -65,10 +96,25 @@
             </visual>
         </link>
+        <joint name="base_sw_top_joint" type = "fixed">
+            <parent link="base_link"/>
+            <child link="swivel_top"/>
+            <origin xyz="0 0 -0.1" rpy="0 0 0"/>
+        </joint>
         <joint name="swivel_joint" type="continuous">
-            <parent link="base_link"/>
-            <child link="spreader_link"/>
-            <origin xyz="0 0 -1" rpy="0 0 0"/>
+            <parent link="swivel_top"/>
+            <child link="swivel_bottom"/>
+            <origin xyz="0 0 -0.1" rpy="0 0 0"/>
             <axis xyz="0 0 1"/>
             <limit effort="100" velocity="1.0"/>
+        </joint>
+        <joint name="swivel_spreader_joint" type="fixed">
+            <parent link="swivel_bottom"/>
+            <child link="spreader_link"/>
+            <origin xyz="0 0 -0.75" rpy="0 0 0"/>
+        </joint>
+        <joint name="swivel_bottom_tag_joint" type="fixed">
+            <parent link="swivel_bottom"/>
+            <child link ="Swivel_Tag"/>
+            <origin xyz ="0.0 0.1 0" rpy="-${pi} 0 ${pi/2}"/>
         </joint>
         <joint name="LG_lin_joint" type="prismatic">
@@ -86,5 +132,5 @@
             <limit lower="0.0" upper="0.5" effort="100" velocity="1.0"/>
         </joint>
-        <joint name="spreader_camera_joint" type="fixed">
+        <joint name="spreader_RS_joint" type="fixed">
             <parent link="spreader_link"/>
             <child link ="Crane_RS_link"/>

Commit message: wheels bringup

File: crane_description/urdf/common.xacro (robot description, xacro)
@@ -20,3 +20,6 @@
         <color rgba="${10/255} ${10/255} ${200/255} 1.0"/>
     </material>
+    <material name= "light_green">
+        <color rgba="${10/255} ${200/255} ${10/255} 1.0"/>
+    </material>
 </robot>

File: crane_description/urdf/crane/crane_macro.ros2_control.xacro (robot description, xacro)
@@ -11,5 +11,5 @@
       <hardware>
         <plugin>crane_hardware/CraneHardware</plugin>
-        <param name="port">/dev/ttyACM1</param>
+        <param name="port">/dev/ttyACM0</param>
         <param name="baud_rate">115200</param>
         <param name="swivel_steps_per_unit">1000.0</param>

File: crane_description/urdf/crane/crane_macro.xacro (robot description, xacro)
@@ -109,12 +109,228 @@
             </visual>
         </link>
-        <link name="Gimbal_0_link"/>
-        <link name="Gimbal_1_link"/>
-        <link name="Gimbal_2_link"/>
-        <link name="Gimbal_3_link"/>
-        <link name="w0_link"/>
-        <link name="w1_link"/>
-        <link name="w2_link"/>
-        <link name="w3_link"/>
+        <link name="Gimbal_0_link">
+            <inertial>
+             <origin
+                xyz="-0.125 -0.028951 0"
+                rpy="0 0 0" />
+            <mass value="1.2749"/>
+            <inertia
+                ixx=".00207"
+                ixy="0"
+                ixz="0"
+                iyy=".005608"
+                iyz="0"
+                izz="0.007147"/>
+            </inertial>
+            <collision>
+            <origin xyz="0 0 0" rpy="0 0 0"/>
+            <geometry>
+                <mesh filename="package://crane_description/meshes/gimbal_0.stl"/>
+            </geometry>
+            </collision>
+            <visual>
+            <origin xyz="0 0 0" rpy="0 0 0"/>
+            <geometry>
+                <mesh filename="package://crane_description/meshes/gimbal_0.stl"/>
+            </geometry>
+            <material name="light_blue"/>
+            </visual>
+        </link>
+        <link name="Gimbal_1_link">
+            <inertial>
+             <origin
+                xyz="-0.028951 0 -0.125"
+                rpy="0 0 0" />
+            <mass value="1.2749"/>
+            <inertia
+                ixx=".005608"
+                ixy="0"
+                ixz="0"
+                iyy="0.007147"
+                iyz="0"
+                izz="0.00207"/>
+            </inertial>
+            <collision>
+            <origin xyz="0 0 0" rpy="0 0 0"/>
+            <geometry>
+                <mesh filename="package://crane_description/meshes/gimbal_12.stl"/>
+            </geometry>
+            </collision>
+            <visual>
+            <origin xyz="0 0 0" rpy="0 0 0"/>
+            <geometry>
+                <mesh filename="package://crane_description/meshes/gimbal_12.stl"/>
+            </geometry>
+            <material name="light_blue"/>
+            </visual>
+        </link>
+        <link name="Gimbal_2_link">
+        <inertial>
+             <origin
+                xyz="-0.028951 0 -0.125"
+                rpy="0 0 0" />
+            <mass value="1.2749"/>
+            <inertia
+                ixx=".005608"
+                ixy="0"
+                ixz="0"
+                iyy="0.007147"
+                iyz="0"
+                izz="0.00207"/>
+            </inertial>
+            <collision>
+            <origin xyz="0 0 0" rpy="0 0 0"/>
+            <geometry>
+                <mesh filename="package://crane_description/meshes/gimbal_12.stl"/>
+            </geometry>
+            </collision>
+            <visual>
+            <origin xyz="0 0 0" rpy="0 0 0"/>
+            <geometry>
+                <mesh filename="package://crane_description/meshes/gimbal_12.stl"/>
+            </geometry>
+            <material name="light_blue"/>
+            </visual>
+        </link>
+        <link name="Gimbal_3_link">
+        <inertial>
+             <origin
+                xyz="-0.125 -0.028951 0"
+                rpy="0 0 0" />
+            <mass value="1.2749"/>
+            <inertia
+                ixx=".00207"
+                ixy="0"
+                ixz="0"
+                iyy=".005608"
+                iyz="0"
+                izz="0.007147"/>
+            </inertial>
+            <collision>
+            <origin xyz="0 0 0" rpy="0 0 0"/>
+            <geometry>
+                <mesh filename="package://crane_description/meshes/gimbal_3.stl"/>
+            </geometry>
+            </collision>
+            <visual>
+            <origin xyz="0 0 0" rpy="0 0 0"/>
+            <geometry>
+                <mesh filename="package://crane_description/meshes/gimbal_3.stl"/>
+            </geometry>
+            <material name="light_blue"/>
+            </visual>
+        </link>
+        <link name="w0_link">
+        <inertial>
+             <origin
+                xyz="0 0 0"
+                rpy="0 0 0" />
+            <mass value="2.0887"/>
+            <inertia
+                ixx=".007176"
+                ixy="0"
+                ixz="0"
+                iyy=".014182"
+                iyz="0"
+                izz="0.007176"/>
+            </inertial>
+            <collision>
+            <origin xyz="0 0 0" rpy="0 0 0"/>
+            <geometry>
+                <mesh filename="package://crane_description/meshes/wheel_03.stl"/>
+            </geometry>
+            </collision>
+            <visual>
+            <origin xyz="0 0 0" rpy="0 0 0"/>
+            <geometry>
+                <mesh filename="package://crane_description/meshes/wheel_03.stl"/>
+            </geometry>
+            <material name="light_green"/>
+            </visual>
+        </link>
+        <link name="w1_link">
+        <inertial>
+             <origin
+                xyz="0 0 0"
+                rpy="0 0 0" />
+            <mass value="2.0887"/>
+            <inertia
+                ixx=".014182"
+                ixy="0"
+                ixz="0"
+                iyy=".007176"
+                iyz="0"
+                izz="0.007176"/>
+            </inertial>
+            <collision>
+            <origin xyz="0 0 0" rpy="0 0 0"/>
+            <geometry>
+                <mesh filename="package://crane_description/meshes/wheel_12.stl"/>
+            </geometry>
+            </collision>
+            <visual>
+            <origin xyz="0 0 0" rpy="0 0 0"/>
+            <geometry>
+                <mesh filename="package://crane_description/meshes/wheel_12.stl"/>
+            </geometry>
+            <material name="light_green"/>
+            </visual>
+        </link>
+        <link name="w2_link">
+        <inertial>
+             <origin
+                xyz="0 0 0"
+                rpy="0 0 0" />
+            <mass value="2.0887"/>
+            <inertia
+                ixx=".014182"
+                ixy="0"
+                ixz="0"
+                iyy=".007176"
+                iyz="0"
+                izz="0.007176"/>
+            </inertial>
+            <collision>
+            <origin xyz="0 0 0" rpy="0 0 0"/>
+            <geometry>
+                <mesh filename="package://crane_description/meshes/wheel_12.stl"/>
+            </geometry>
+            </collision>
+            <visual>
+            <origin xyz="0 0 0" rpy="0 0 0"/>
+            <geometry>
+                <mesh filename="package://crane_description/meshes/wheel_12.stl"/>
+            </geometry>
+            <material name="light_green"/>
+            </visual>
+        </link>
+        <link name="w3_link">
+        <inertial>
+             <origin
+                xyz="0 0 0"
+                rpy="0 0 0" />
+            <mass value="2.0887"/>
+            <inertia
+                ixx=".007176"
+                ixy="0"
+                ixz="0"
+                iyy=".014182"
+                iyz="0"
+                izz="0.007176"/>
+            </inertial>
+            <collision>
+            <origin xyz="0 0 0" rpy="0 0 0"/>
+            <geometry>
+                <mesh filename="package://crane_description/meshes/wheel_03.stl"/>
+            </geometry>
+            </collision>
+            <visual>
+            <origin xyz="0 0 0" rpy="0 0 0"/>
+            <geometry>
+                <mesh filename="package://crane_description/meshes/wheel_03.stl"/>
+            </geometry>
+            <material name="light_green"/>
+            </visual>
+        </link>
         <joint name="base_sw_top_joint" type = "fixed">
             <parent link="base_link"/>
